Commit message: Modify get_object_positions

File: urdf/kitchen/yellow_bowl/model.urdf (robot description, URDF)
Before this commit: robot Cole_Hardware_Bowl_Scirocco_YellowBlue, 1 links, 0 joints
Links:
- link link_0: geometry collision mesh filename=meshes/model.obj; visual mesh filename=meshes/model.obj
