Commit message: add self-made urdf

File: urdf/robot/ur_description/eugene_robot_2fg7.urdf (robot description, URDF)
Before this commit: robot ur5e, 14 links, 13 joints
Links:
- removed link ur10_leftfinger_ft_sensor
- removed link ur10_rightfinger_ft_sensor
- added link ur_leftfinger_ft_sensor; collision box size=0.01 0.02 0.0005; visual box size=0.01 0.02 0.0005
- added link ur_rightfinger_ft_sensor; collision box size=0.020 0.01 0.0005; visual box size=0.020 0.01 0.0005
- link hand_link: geometry visual mesh filename=meshes/onrobot_2fg7_description/meshes/base_link.stl scale=0.001 0.001 0.001
Joints:
- removed joint ur10_leftfinger_ft_sensor_joint
- removed joint ur10_rightfinger_ft_sensor_joint
- added joint ur_leftfinger_ft_sensor_joint: type fixed, parent left_finger_link, child ur_leftfinger_ft_sensor, origin xyz=0.003847703322119739 0.029496959480080673 0.032234215486237948 rpy=0 -1.57 0
- added joint ur_rightfinger_ft_sensor_joint: type fixed, parent right_finger_link, child ur_rightfinger_ft_sensor, origin xyz=0.018274296677847158 0.029496959480080673 0.032234215486237948 rpy=0 -1.57 0
- joint gripper_center_joint: origin xyz=0.1525 0.0 0.0 rpy=0.00000 0.00000 0.00000 -> xyz=0.155 0.0 0.0 rpy=0.00000 0.00000 0.00000
